Commit message: add 3D Lidar VLP16 and 4D Lidar L1

File: unitree_go2_description/urdf/unitree_go2_robot.xacro (robot description, xacro)
@@ -8,4 +8,6 @@
     <xacro:include filename="$(find unitree_go2_description)/urdf/unitree_go2_gazebo.xacro"/>
     <!-- <xacro:include filename="$(find unitree_go2_description)/launch/stairs.urdf.xacro"/> -->
+    <xacro:include filename="$(find unitree_go2_description)/urdf/velodyne.xacro"/>
+    <xacro:include filename="$(find unitree_go2_description)/urdf/lidar_4D_lidar.xacro"/>
     <!-- <xacro:stairs stairs="15" xpos="0" ypos="0" zpos="0" /> -->
     <!-- Rotor related joint and link is only for demonstrate location. -->
@@ -39,5 +41,4 @@
                 <mesh filename="file://$(find unitree_go2_description)/meshes/trunk.dae" scale="1 1 1"/>
             </geometry>
-            <!-- <material name="orange"/> -->
         </visual>
         <collision>
@@ -80,30 +81,34 @@
         </collision>
     </link>
-    <!--
-    <joint name="load_joint" type="fixed">
-        <parent link="trunk"/>
-        <child link="load_link"/>
-        <origin rpy="0 0 0" xyz="0 0 0"/>
+    <!-- <joint name="lidar_l1_joint" type="fixed">
+        <parent link="base_link"/>
+        <child link="lidar_l1_link"/>
+        <origin rpy="2.94 0 1.5705" xyz="0.25 -0.038 -0.03"/>
     </joint>
-    <link name="load_link">
+    <link name="lidar_l1_link">
         <inertial>
-            <mass value="5"/>
+            <mass value="0.5"/>
             <origin rpy="0 0 0" xyz="0 0 0"/>
             <inertia ixx="0.01" ixy="0" ixz="0" iyy="0.01" iyz="0" izz="0.01"/>
         </inertial>
         <visual>
-            <origin rpy="0 0 0" xyz="0 0 0.2"/>
+            <origin rpy="0 0 0" xyz="0 0 0"/>
             <geometry>
-                <box size="0.5 0.3 0.2"/>
+                <mesh filename="file://$(find unitree_go2_description)/meshes/L1_4D_Lidar.dae" scale="1 1 1"/>
             </geometry>
+            <material name="black">
+                <color rgba="0.0 0.0 0.0 1.0"/>
+            </material>
         </visual>
         <collision>
             <origin rpy="0 0 0" xyz="0 0 0"/>
             <geometry>
-                <box size=".001 .001 .001"/>
+                <mesh filename="file://$(find unitree_go2_description)/meshes/L1_4D_Lidar.dae" scale="1 1 1"/>
             </geometry>
+            <material name="black">
+                <color rgba="0.0 0.0 0.0 1.0"/>
+            </material>
         </collision>
-    </link>
--->
+    </link> -->
     <xacro:leg name="rf" mirror="-1" mirror_dae= "False" front_hind="1"  front_hind_dae="True"  />
     <xacro:leg name="lf" mirror="1"  mirror_dae="True"   front_hind="1"  front_hind_dae="True"  />
