Commit message: add Mono Camera

File: unitree_go2_description/urdf/unitree_go2_gazebo.xacro (robot description, xacro)
@@ -1,147 +1,169 @@
 <?xml version="1.0"?>
 <robot>
-    <!-- Gazebo Sim plugins -->
-    <gazebo>
-      <plugin filename="gz-sim-pose-publisher-system" name="gz::sim::systems::PosePublisher">
-        <publish_link_pose>true</publish_link_pose>
-        <publish_sensor_pose>true</publish_sensor_pose>
-        <publish_collision_pose>false</publish_collision_pose>
-        <publish_visual_pose>false</publish_visual_pose>
-        <publish_nested_model_pose>false</publish_nested_model_pose>
-        <use_pose_vector_msg>true</use_pose_vector_msg>
-        <static_publisher>true</static_publisher>
-        <static_update_frequency>100</static_update_frequency>
+  <!-- Gazebo Sim plugins -->
+  <gazebo>
+    <plugin filename="gz-sim-pose-publisher-system" name="gz::sim::systems::PosePublisher">
+      <publish_link_pose>true</publish_link_pose>
+      <publish_sensor_pose>true</publish_sensor_pose>
+      <publish_collision_pose>false</publish_collision_pose>
+      <publish_visual_pose>false</publish_visual_pose>
+      <publish_nested_model_pose>false</publish_nested_model_pose>
+      <use_pose_vector_msg>true</use_pose_vector_msg>
+      <static_publisher>true</static_publisher>
+      <static_update_frequency>100</static_update_frequency>
+    </plugin>
+  </gazebo>
+  <!-- Robot-wide physics properties -->
+  <gazebo>
+    <plugin filename="gz-sim-physics-system" name="gz::sim::systems::Physics">
+      <engine>
+        <filename>gz-physics-ode-plugin</filename>
+      </engine>
+    </plugin>
+  </gazebo>
+  <!-- ROS2 Control plugin -->
+  <gazebo>
+    <plugin filename="gz_ros2_control-system" name="gz_ros2_control::GazeboSimROS2ControlPlugin">
+      <parameters>$(find unitree_go2_sim)/config/ros_control/ros_control.yaml</parameters>
+      <robot_param_node>robot_state_publisher</robot_param_node>
+    </plugin>
+  </gazebo>
+  <!-- IMU plugin -->
+  <gazebo reference="imu_link">
+    <sensor name="imu_sensor" type="imu">
+      <always_on>true</always_on>
+      <update_rate>100</update_rate>
+      <visualize>true</visualize>
+      <topic>imu</topic>
+      <gz_frame_id>imu_link</gz_frame_id>
+      <plugin filename="gz-sim-imu-system" name="gz::sim::systems::Imu">
+        <initial_orientation_as_reference>false</initial_orientation_as_reference>
       </plugin>
-    </gazebo>
-    <!-- Robot-wide physics properties -->
-    <gazebo>
-      <plugin filename="gz-sim-physics-system" name="gz::sim::systems::Physics">
-        <engine>
-          <filename>gz-physics-ode-plugin</filename>
-        </engine>
-      </plugin>
-    </gazebo>
-    <!-- ROS2 Control plugin -->
-    <gazebo>
-      <plugin filename="gz_ros2_control-system" name="gz_ros2_control::GazeboSimROS2ControlPlugin">
-        <parameters>$(find unitree_go2_sim)/config/ros_control/ros_control.yaml</parameters>
-        <robot_param_node>robot_state_publisher</robot_param_node>
-      </plugin>
-    </gazebo>
-    <!-- IMU plugin -->
-    <gazebo reference="imu_link">
-      <sensor name="imu_sensor" type="imu">
-        <always_on>true</always_on>
-        <update_rate>100</update_rate>
-        <visualize>true</visualize>
-        <topic>imu</topic>
-        <gz_frame_id>imu_link</gz_frame_id>
-        <plugin filename="gz-sim-imu-system" name="gz::sim::systems::Imu">
-          <initial_orientation_as_reference>false</initial_orientation_as_reference>
-        </plugin>
-      </sensor>
-    </gazebo>
-    <!-- Main body -->
-    <gazebo reference="trunk">
-      <mu1>0.2</mu1>
-      <mu2>0.2</mu2>
-      <kp>10000.0</kp>
-      <kd>1.0</kd>
-    </gazebo>
-    <!-- FL leg -->
-    <gazebo reference="lf_hip_link">
-      <mu1>0.2</mu1>
-      <mu2>0.2</mu2>
-    </gazebo>
-    <gazebo reference="lf_upper_leg_link">
-      <mu1>0.2</mu1>
-      <mu2>0.2</mu2>
-      <self_collide>1</self_collide>
-      <kp>10000.0</kp>
-      <kd>1.0</kd>
-    </gazebo>
-    <gazebo reference="lf_lower_leg_link">
-      <mu1>0.2</mu1>
-      <mu2>0.2</mu2>
-      <self_collide>1</self_collide>
-    </gazebo>
-    <gazebo reference="lf_foot_link">
-      <mu1>0.6</mu1>
-      <mu2>0.6</mu2>
-      <self_collide>1</self_collide>
-      <kp>10000.0</kp>
-      <kd>1.0</kd>
-    </gazebo>
-    <!-- FR leg -->
-    <gazebo reference="rf_hip_link">
-      <mu1>0.2</mu1>
-      <mu2>0.2</mu2>
-    </gazebo>
-    <gazebo reference="rf_upper_leg_link">
-      <mu1>0.2</mu1>
-      <mu2>0.2</mu2>
-      <self_collide>1</self_collide>
-      <kp>10000.0</kp>
-      <kd>1.0</kd>
-    </gazebo>
-    <gazebo reference="rf_lower_leg_link">
-      <mu1>0.2</mu1>
-      <mu2>0.2</mu2>
-      <self_collide>1</self_collide>
-    </gazebo>
-    <gazebo reference="rf_foot_link">
-      <mu1>0.6</mu1>
-      <mu2>0.6</mu2>
-      <self_collide>1</self_collide>
-      <kp>10000.0</kp>
-      <kd>1.0</kd>
-    </gazebo>
-    <!-- RL leg -->
-    <gazebo reference="lh_hip_link">
-      <mu1>0.2</mu1>
-      <mu2>0.2</mu2>
-    </gazebo>
-    <gazebo reference="lh_upper_leg_link">
-      <mu1>0.2</mu1>
-      <mu2>0.2</mu2>
-      <self_collide>1</self_collide>
-      <kp>10000.0</kp>
-      <kd>1.0</kd>
-    </gazebo>
-    <gazebo reference="lh_lower_leg_link">
-      <mu1>0.2</mu1>
-      <mu2>0.2</mu2>
-      <self_collide>1</self_collide>
-    </gazebo>
-    <gazebo reference="lh_foot_link">
-      <mu1>0.6</mu1>
-      <mu2>0.6</mu2>
-      <self_collide>1</self_collide>
-      <kp>10000.0</kp>
-      <kd>1.0</kd>
-    </gazebo>
-    <!-- RR leg -->
-    <gazebo reference="rh_hip_link">
-      <mu1>0.2</mu1>
-      <mu2>0.2</mu2>
-    </gazebo>
-    <gazebo reference="rh_upper_leg_link">
-      <mu1>0.2</mu1>
-      <mu2>0.2</mu2>
-      <self_collide>1</self_collide>
-      <kp>10000.0</kp>
-      <kd>1.0</kd>
-    </gazebo>
-    <gazebo reference="rh_lower_leg_link">
-      <mu1>0.2</mu1>
-      <mu2>0.2</mu2>
-      <self_collide>1</self_collide>
-    </gazebo>
-    <gazebo reference="rh_foot_link">
-      <mu1>0.6</mu1>
-      <mu2>0.6</mu2>
-      <self_collide>1</self_collide>
-      <kp>10000.0</kp>
-      <kd>1.0</kd>
-    </gazebo>
+    </sensor>
+  </gazebo>
+  <!-- Camera Plugin-->
+  <gazebo reference="camera_link">
+    <sensor name="rgb_camera" type="camera">
+      <pose>0 0.0 0 0 0 0</pose>
+      <camera>
+        <horizontal_fov>1.367</horizontal_fov>
+        <image>
+          <width>640</width>
+          <height>480</height>
+        </image>
+        <clip>
+          <near>0.05</near>
+          <far>200</far>
+        </clip>
+      </camera>
+      <gz_frame_id>camera_link</gz_frame_id>
+      <always_on>1</always_on>
+      <update_rate>10</update_rate>
+      <visualize>1</visualize>
+      <topic>rgb_image</topic>
+    </sensor>
+  </gazebo>
+  <!-- Main body -->
+  <gazebo reference="trunk">
+    <mu1>0.2</mu1>
+    <mu2>0.2</mu2>
+    <kp>10000.0</kp>
+    <kd>1.0</kd>
+  </gazebo>
+  <!-- FL leg -->
+  <gazebo reference="lf_hip_link">
+    <mu1>0.2</mu1>
+    <mu2>0.2</mu2>
+  </gazebo>
+  <gazebo reference="lf_upper_leg_link">
+    <mu1>0.2</mu1>
+    <mu2>0.2</mu2>
+    <self_collide>1</self_collide>
+    <kp>10000.0</kp>
+    <kd>1.0</kd>
+  </gazebo>
+  <gazebo reference="lf_lower_leg_link">
+    <mu1>0.2</mu1>
+    <mu2>0.2</mu2>
+    <self_collide>1</self_collide>
+  </gazebo>
+  <gazebo reference="lf_foot_link">
+    <mu1>0.6</mu1>
+    <mu2>0.6</mu2>
+    <self_collide>1</self_collide>
+    <kp>10000.0</kp>
+    <kd>1.0</kd>
+  </gazebo>
+  <!-- FR leg -->
+  <gazebo reference="rf_hip_link">
+    <mu1>0.2</mu1>
+    <mu2>0.2</mu2>
+  </gazebo>
+  <gazebo reference="rf_upper_leg_link">
+    <mu1>0.2</mu1>
+    <mu2>0.2</mu2>
+    <self_collide>1</self_collide>
+    <kp>10000.0</kp>
+    <kd>1.0</kd>
+  </gazebo>
+  <gazebo reference="rf_lower_leg_link">
+    <mu1>0.2</mu1>
+    <mu2>0.2</mu2>
+    <self_collide>1</self_collide>
+  </gazebo>
+  <gazebo reference="rf_foot_link">
+    <mu1>0.6</mu1>
+    <mu2>0.6</mu2>
+    <self_collide>1</self_collide>
+    <kp>10000.0</kp>
+    <kd>1.0</kd>
+  </gazebo>
+  <!-- RL leg -->
+  <gazebo reference="lh_hip_link">
+    <mu1>0.2</mu1>
+    <mu2>0.2</mu2>
+  </gazebo>
+  <gazebo reference="lh_upper_leg_link">
+    <mu1>0.2</mu1>
+    <mu2>0.2</mu2>
+    <self_collide>1</self_collide>
+    <kp>10000.0</kp>
+    <kd>1.0</kd>
+  </gazebo>
+  <gazebo reference="lh_lower_leg_link">
+    <mu1>0.2</mu1>
+    <mu2>0.2</mu2>
+    <self_collide>1</self_collide>
+  </gazebo>
+  <gazebo reference="lh_foot_link">
+    <mu1>0.6</mu1>
+    <mu2>0.6</mu2>
+    <self_collide>1</self_collide>
+    <kp>10000.0</kp>
+    <kd>1.0</kd>
+  </gazebo>
+  <!-- RR leg -->
+  <gazebo reference="rh_hip_link">
+    <mu1>0.2</mu1>
+    <mu2>0.2</mu2>
+  </gazebo>
+  <gazebo reference="rh_upper_leg_link">
+    <mu1>0.2</mu1>
+    <mu2>0.2</mu2>
+    <self_collide>1</self_collide>
+    <kp>10000.0</kp>
+    <kd>1.0</kd>
+  </gazebo>
+  <gazebo reference="rh_lower_leg_link">
+    <mu1>0.2</mu1>
+    <mu2>0.2</mu2>
+    <self_collide>1</self_collide>
+  </gazebo>
+  <gazebo reference="rh_foot_link">
+    <mu1>0.6</mu1>
+    <mu2>0.6</mu2>
+    <self_collide>1</self_collide>
+    <kp>10000.0</kp>
+    <kd>1.0</kd>
+  </gazebo>
 </robot>

File: unitree_go2_description/urdf/unitree_go2_robot.xacro (robot description, xacro)
@@ -1,4 +1,5 @@
 <?xml version="1.0"?>
-<robot name="go2" xmlns:xacro="http://www.ros.org/wiki/xacro">
+<robot name="go2"
+    xmlns:xacro="http://www.ros.org/wiki/xacro">
     <xacro:arg name="DEBUG" default="false"/>
     <xacro:include filename="$(find unitree_go2_description)/urdf/const.xacro"/>
@@ -51,8 +52,5 @@
             <origin rpy="0 0 0" xyz="${trunk_com_x} ${trunk_com_y} ${trunk_com_z}"/>
             <mass value="${trunk_mass}"/>
-            <inertia
-                ixx="${trunk_ixx}" ixy="${trunk_ixy}" ixz="${trunk_ixz}"
-                iyy="${trunk_iyy}" iyz="${trunk_iyz}"
-                izz="${trunk_izz}"/>
+            <inertia ixx="${trunk_ixx}" ixy="${trunk_ixy}" ixz="${trunk_ixz}" iyy="${trunk_iyy}" iyz="${trunk_iyz}" izz="${trunk_izz}"/>
         </inertial>
     </link>
@@ -81,4 +79,32 @@
         </collision>
     </link>
+    <!-- Camera Link-->
+    <link name="camera_link">
+        <inertial>
+            <mass value="0.001"/>
+            <origin rpy="0 0 0" xyz="0 0 0"/>
+            <inertia ixx="0.0001" ixy="0" ixz="0" iyy="0.0001" iyz="0" izz="0.0001"/>
+        </inertial>
+        <visual>
+            <origin rpy="0 0 0" xyz="0 0 0"/>
+            <geometry>
+                <sphere radius="0.001"/>
+            </geometry>
+            <material name="">
+                <color rgba="0.5 0 0 1" />
+            </material>
+        </visual>
+        <collision>
+            <origin rpy="0 0 0" xyz="0 0 0"/>
+            <geometry>
+                <sphere radius="0.001"/>
+            </geometry>
+        </collision>
+    </link>
+    <joint name="camera_joint" type="fixed">
+        <parent link="trunk"/>
+        <child link="camera_link"/>
+        <origin rpy="0 0 0" xyz="0.326 0 0.043"/>
+    </joint>
     <!-- <joint name="lidar_l1_joint" type="fixed">
         <parent link="base_link"/>
@@ -111,7 +137,7 @@
         </collision>
     </link> -->
-    <xacro:leg name="rf" mirror="-1" mirror_dae= "False" front_hind="1"  front_hind_dae="True"  />
-    <xacro:leg name="lf" mirror="1"  mirror_dae="True"   front_hind="1"  front_hind_dae="True"  />
-    <xacro:leg name="rh" mirror="-1" mirror_dae="False"  front_hind="-1" front_hind_dae="False" />
-    <xacro:leg name="lh" mirror="1"  mirror_dae="True"   front_hind="-1" front_hind_dae="False" />
+    <xacro:leg name="rf" mirror="-1" mirror_dae= "False" front_hind="1" front_hind_dae="True" />
+    <xacro:leg name="lf" mirror="1" mirror_dae="True" front_hind="1" front_hind_dae="True" />
+    <xacro:leg name="rh" mirror="-1" mirror_dae="False" front_hind="-1" front_hind_dae="False" />
+    <xacro:leg name="lh" mirror="1" mirror_dae="True" front_hind="-1" front_hind_dae="False" />
 </robot>
